Commit message: Basic planning working

File: urdf/dual_arm_husky.urdf.xacro (robot description, xacro)
@@ -11,5 +11,5 @@
     <xacro:include filename="$(find ur_description)/urdf/ur_macro.xacro"/>
     <!-- convert to property to use substitution in function -->
-    <xacro:property name="initial_positions_file" default="$(find ur_description)/config/initial_positions.yaml"/>
+    <xacro:property name="initial_positions_file" default="$(find dual_arm_husky_description)/config/${prefix}initial_positions.yaml"/>
     <!-- arm -->
     <xacro:ur_robot
@@ -21,6 +21,6 @@
       physical_parameters_file="$(find ur_description)/config/${ur_type}/physical_parameters.yaml"
       visual_parameters_file="$(find ur_description)/config/${ur_type}/visual_parameters.yaml"
-      use_fake_hardware="true"
-      fake_sensor_commands="true"
+      use_fake_hardware="false"
+      fake_sensor_commands="false"
       sim_gazebo="false"
       sim_ignition="true"
@@ -72,9 +72,9 @@
   <gazebo reference="world"/>
   <gazebo>
-      <plugin filename="libign_ros2_control-system.so" name="ign_ros2_control::IgnitionROS2ControlPlugin">
-        <robot_param>robot_description</robot_param>
-        <robot_param_node>robot_state_publisher</robot_param_node>
-        <parameters>$(find dual_arm_husky_description)/config/controllers.yaml</parameters>
-      </plugin>
+    <plugin filename="libign_ros2_control-system.so" name="ign_ros2_control::IgnitionROS2ControlPlugin">
+      <robot_param>robot_description</robot_param>
+      <robot_param_node>robot_state_publisher</robot_param_node>
+      <parameters>$(find dual_arm_husky_description)/config/controllers.yaml</parameters>
+    </plugin>
   </gazebo>
   <!-- <world>
